File: BoxTurtleMC.kicad_pcb (KiCad board)
At the start: 2 copper layers, 110 x 60 mm, 35 parts, among them M1 Conn_01x02 Pin1+ Pin2-, M2 Conn_01x02 Pin1+ Pin2-, M3 Conn_01x02 Pin1+ Pin2-, M4 Conn_01x02 Pin1+ Pin2-, M5 Conn_01x02 Pin1+ Pin2-, M6 Conn_01x02 Pin1+ Pin2-, M7 Conn_01x02 Pin1+ Pin2-, M8 Conn_01x02 Pin1+ Pin2-, SW1 Conn_01x02 Pin1+ Pin2-, SW2 Conn_01x02 Pin1+ Pin2-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

Commit message: Added notes about using with Ender 3 SKR board.
Other:
- board text added: "BoxTurtleMC v1.1.1"
- board text added: "GP12"
- board text added: "SW7"
- board text removed: "BoxTurtleMC v1.1"
Changed lines of the file:
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@@
 		)
 		(fp_text user "DRV8833"
-			(at -6.25 -4.25 90)
+			(at -6.375 3.8857 90)
 			(unlocked yes)
 			(layer "F.SilkS")
@@
 		)
 		(fp_text user "IN3"
-			(at 6.25 -3.25 90)
+			(at 6.225 -3.1143 90)
 			(unlocked yes)
 			(layer "B.SilkS")
@@
 		(net 1)
 	)
+	(gr_rect
+		(start 159.5 106.25)
+		(end 160.1 106.3)
+		(stroke
+			(width 0.15)
+			(type default)
+		)
+		(fill no)
+		(layer "F.SilkS")
+	)
+	(gr_rect
+		(start 159.5 103.9)
+		(end 161 104.5)
+		(stroke
+			(width 0.15)
+			(type default)
+		)
+		(fill no)
+		(layer "F.SilkS")
+	)
+	(gr_rect
+		(start 161.75 103.9)
+		(end 162.25 104.5)
+		(stroke
+			(width 0.15)
+			(type default)
+		)
+		(fill no)
+		(layer "F.SilkS")
+	)
+	(gr_rect
+		(start 160.1 108.1)
+		(end 163.8 108.1)
+		(stroke
+			(width 0.15)
+			(type default)
+		)
+		(fill no)
+		(layer "F.SilkS")
+	)
+	(gr_rect
+		(start 163.9 106.3)
+		(end 163.9 108.1)
+		(stroke
+			(width 0.15)
+			(type default)
+		)
+		(fill no)
+		(layer "F.SilkS")
+	)
+	(gr_rect
+		(start 159.5 103.9)
+		(end 164.5 108.6)
+		(stroke
+			(width 0.15)
+			(type default)
+		)
+		(fill no)
+		(layer "F.SilkS")
+	)
+	(gr_rect
+		(start 163.9 106.25)
+		(end 164.5 106.3)
+		(stroke
+			(width 0.15)
+			(type default)
+		)
+		(fill no)
+		(layer "F.SilkS")
+	)
+	(gr_rect
+		(start 163.1 103.9)
+		(end 164.5 104.5)
+		(stroke
+			(width 0.15)
+			(type default)
+		)
+		(fill no)
+		(layer "F.SilkS")
+	)
+	(gr_rect
+		(start 160.1 106.3)
+		(end 160.1 108.1)
+		(stroke
+			(width 0.15)
+			(type default)
+		)
+		(fill no)
+		(layer "F.SilkS")
+	)
 	(gr_line
 		(start 116.85 89.35)
@@
 		)
 	)
-	(gr_text "BoxTurtleMC v1.1"
+	(gr_text "BoxTurtleMC v1.1.1"
 		(at 144.7 74 0)
 		(layer "F.SilkS")
@@
 		)
 	)
+	(gr_text "SW7"
+		(at 162 110.8 0)
+		(layer "F.SilkS")
+		(effects
+			(font
+				(size 1 1)
+				(thickness 0.15)
+			)
+		)
+	)
 	(gr_text "GND"
 		(at 165.8 86.8 0)
@@
 		)
 	)
+	(gr_text "GP12"
+		(at 158.5 109.8 0)
+		(layer "F.SilkS")
+		(effects
+			(font
+				(size 0.8 0.8)
+				(thickness 0.1)
+			)
+			(justify left bottom)
+		)
+	)
+	(gr_text "GND"
+		(at 162.8 109.8 0)
+		(layer "F.SilkS")
+		(effects
+			(font
+				(size 0.8 0.8)
+				(thickness 0.1)
+			)
+			(justify left bottom)
+		)
+	)
 	(gr_text "-"
 		(at 144.55 124.2765 0)
@@
 		)
 	)
-	(gr_text "BoxTurtleMC v1.1"
+	(gr_text "BoxTurtleMC v1.1.1"
 		(at 171.95 74 0)
 		(layer "B.SilkS")

Commit message: Update to version 1.1.2
Parts:
- added JP3: SolderJumper_2_Bridged, Jumper:SolderJumper-2_P1.3mm_Bridged_RoundedPad1.0x1.5mm, F.Cu at (170.5, 85.0)
- added JP4: SolderJumper_2_Bridged, Jumper:SolderJumper-2_P1.3mm_Bridged_RoundedPad1.0x1.5mm, F.Cu at (177.1, 85.0)
- added SW7: Conn_01x02 Pin1+ Pin2-, Connector_JST:JST_XH_B2B-XH-A_1x02_P2.50mm_Vertical, F.Cu at (165.7, 74.8)
- added SW8: Conn_01x02 Pin1+ Pin2-, Connector_JST:JST_XH_B2B-XH-A_1x02_P2.50mm_Vertical, F.Cu at (174.2, 74.8)
- moved JP1 19.6 mm to (157.5, 85.0)
- moved SW6 16.2 mm to (157.2, 74.8), turned to 0 degrees
- moved SW5 15.5 mm to (148.7, 74.8), turned to 0 degrees
- moved JP2 12.8 mm to (164.1, 85.0)
- renumbered JP2 to JP1, JP1 to JP2
Connections:
- U2 pad 19: Net-(DRV4-AIN1) -> Net-(JP4-B)
- U2 pad 20: Net-(DRV4-AIN2) -> Net-(JP3-B)
Routing:
- net GND: track 259.4 -> 343.7 mm
- net Net-(JP4-B): track 0.00 -> 74.4 mm, vias 0 -> 3
- net Net-(JP3-B): track 0.00 -> 31.4 mm, vias 0 -> 3
- net Net-(DRV4-BIN2): track 20.8 -> 38.4 mm
- net +5V: track 136.4 -> 153.7 mm, vias 2 -> 1
- net Net-(DRV4-BIN1): track 27.8 -> 42.7 mm
- net Net-(JP1-B): track 26.5 -> 16.8 mm, vias 1 -> 0
- net Net-(JP2-B): track 32.1 -> 24.4 mm
- net Net-(3.3V1-Pin_1): track 74.6 -> 80.6 mm
- net Net-(120J1-B): track 137.7 -> 132.4 mm
- net Net-(DRV3-AIN2): track 37.9 -> 43.1 mm
- net Net-(D1-K): track 11.4 -> 16.3 mm
- net Net-(DRV4-AIN2): track 42.2 -> 39.0 mm
- net Net-(CAN1-CANL): track 133.2 -> 136.2 mm
- net Net-(SW2-Pin_1): track 9.92 -> 12.6 mm
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Other:
- board text added: "BoxTurtleMC v1.1.2"
- board text added: "GP14"
- board text added: "GP15"
- board text added: "SW9"
- board text removed: "BoxTurtleMC v1.1.1"
- board text removed: "SW7"
