File: BoxTurtleMC.kicad_sch (KiCad schematic)
At the start: 35 parts, among them M1 Conn_01x02 Pin1+ Pin2-, M2 Conn_01x02 Pin1+ Pin2-, M3 Conn_01x02 Pin1+ Pin2-, M4 Conn_01x02 Pin1+ Pin2-, M5 Conn_01x02 Pin1+ Pin2-, M6 Conn_01x02 Pin1+ Pin2-, M7 Conn_01x02 Pin1+ Pin2-, M8 Conn_01x02 Pin1+ Pin2-, SW1 Conn_01x02 Pin1+ Pin2-, SW2 Conn_01x02 Pin1+ Pin2-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

Commit message: Update to version 1.1.2
Parts:
- added JP3, JP4: SolderJumper_2_Bridged, Jumper:SolderJumper-2_P1.3mm_Bridged_RoundedPad1.0x1.5mm, symbol Jumper:SolderJumper_2_Bridged
- added SW7, SW8: Conn_01x02 Pin1+ Pin2-, Connector_JST:JST_XH_B2B-XH-A_1x02_P2.50mm_Vertical, symbol Connector_Generic:Conn_01x02
- renumbered JP2 to JP1, JP1 to JP2
Connections:
- net GND: now also SW7.2 (Pin_2), SW8.2 (Pin_2)
- net at U2.19 (GPIO14): now also JP4.2 (B), SW8.1 (Pin_1); no longer DRV4.7 (AIN1)
- net at U2.20 (GPIO15): now also JP3.2 (B), SW7.1 (Pin_1); no longer DRV4.8 (AIN2)
- new net: DRV4.7 (AIN1), JP4.1 (A)
- new net: DRV4.8 (AIN2), JP3.1 (A)
